File: OneAvionics.kicad_pcb (KiCad board)
At the start: 2 copper layers, 33 x 40.6 mm, 57 parts, among them J1 Conn_01x02, J2 USB_B_Micro, J3 SWD, J4 Micro_SD_Card, J5 ST_01x02, Q1 DMN2230U, SW1 SW_SPDT, SW2 SW_SPDT, SW3 SW_Push, SW4 SW_Push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

Commit message: bno055 removed, bmi088, schotksy
Parts:
- removed C1, C12, C13, C15, C16, C19, C2, C20, C21, C3, C4, C5, C6, C7: 100nF, Capacitor_SMD:C_0603_1608Metric
- removed C10, C11: 22pF, Capacitor_SMD:C_0603_1608Metric
- removed C17: 6.8nF, Capacitor_SMD:C_0603_1608Metric
- removed C18: 120nF, Capacitor_SMD:C_0603_1608Metric
- removed C8: 10uF, Capacitor_SMD:C_0603_1608Metric
- removed C9: 0.1uF, Capacitor_SMD:C_0603_1608Metric
- removed D1: WS2812B, LED_SMD:LED_WS2812B_PLCC4_5.0x5.0mm_P3.2mm
- removed D2, D3: LED, LED_SMD:LED_0805_2012Metric
- removed F1: 2A, Fuse:Fuse_1206_3216Metric_Castellated
- removed H1, H2, H3, H4: MountingHole, MountingHole:MountingHole_2.2mm_M2_Pad_Via
- removed J1: Conn_01x02, TerminalBlock_Phoenix:TerminalBlock_Phoenix_PT-1,5-2-3.5-H_1x02_P3.50mm_Horizontal
- removed J2: USB_B_Micro, Connector_USB:USB_Micro-B_Molex_47346-0001
- removed J3: SWD, Connector_PinHeader_2.54mm:PinHeader_2x05_P2.54mm_Vertical
- removed J4: Micro_SD_Card, Connector_Card:microSD_HC_Hirose_DM3AT-SF-PEJM5
- removed J5: ST_01x02, TerminalBlock_Phoenix:TerminalBlock_Phoenix_PT-1,5-2-3.5-H_1x02_P3.50mm_Horizontal
- removed Q1: DMN2230U, Package_TO_SOT_SMD:SOT-23
- removed R1, R12, R13, R14, R2, R4, R7, R8: 10K, Capacitor_SMD:C_0603_1608Metric
- removed R10, R11, R9: 150R, Capacitor_SMD:C_0603_1608Metric
- removed R3, R6: 22R, Capacitor_SMD:C_0603_1608Metric
- removed R5: 3.8k, Capacitor_SMD:C_0603_1608Metric
- removed SW1, SW2: SW_SPDT, Button_Switch_SMD:SW_SPDT_PCM12
- removed SW3, SW4: SW_Push, Button_Switch_SMD:SW_SPST_B3U-1000P
- removed U1: STM32F103C8Tx, Package_QFP:LQFP-48_7x7mm_P0.5mm
- removed U2: BNO055, Package_LGA:LGA-28_5.2x3.8mm_P0.5mm
- removed U3: LM1117-3.3, Package_TO_SOT_SMD:SOT-223
- removed U4: BMP280, Package_LGA:Bosch_LGA-8_2x2.5mm_P0.65mm_ClockwisePinNumbering
- removed Y1: 16MHz, Crystal:Crystal_SMD_3225-4Pin_3.2x2.5mm
Routing:
- removed copper zone on F.Cu, net +3V3
Other:
- board outline removed
- board text removed: "+"
- board text removed: "+BATT(12V)"
- board text removed: "0"
- board text removed: "1"
- board text removed: "10"
- board text removed: "BOOT0"
- board text removed: "BTN"
- board text removed: "Djino van Dorland"
- board text removed: "ONE"
- board text removed: "PYRO 1"
- board text removed: "RESET"
- board text removed: "SWD"

Commit message: more cleanup
Parts:
- added C1: 100nF, Capacitor_SMD:C_0603_1608Metric, F.Cu at (128.5, 75.8)
- added C10: 22pF, Capacitor_SMD:C_0603_1608Metric, F.Cu at (132.6, 70.8)
- added C11: 22pF, Capacitor_SMD:C_0603_1608Metric, F.Cu at (124.0, 78.8)
- added C12: 100nF, Capacitor_SMD:C_0603_1608Metric, F.Cu at (176.6, 71.4)
- added C13: 100nF, Capacitor_SMD:C_0603_1608Metric, F.Cu at (186.8, 61.6)
- added C14: 10uF, Capacitor_SMD:C_0603_1608Metric, F.Cu at (115.0, 85.5)
- added C15: 100nF, Capacitor_SMD:C_0603_1608Metric, F.Cu at (102.3, 101.0)
- added C16: 100nF, Capacitor_SMD:C_0603_1608Metric, F.Cu at (106.7, 93.5)
- added C17: 100nF, Capacitor_SMD:C_0603_1608Metric, F.Cu at (102.3, 98.5)
- added C19: 100nF, Capacitor_SMD:C_0603_1608Metric, F.Cu at (98.3, 98.6)
- added C2: 100nF, Capacitor_SMD:C_0603_1608Metric, F.Cu at (124.0, 81.3)
- added C21: 100nF, Capacitor_SMD:C_0603_1608Metric, F.Cu at (102.7, 96.0)
- added C22: 0.1uF, Capacitor_SMD:C_0603_1608Metric, F.Cu at (99.6, 69.2)
- added C23: 470uF, Capacitor_SMD:C_0603_1608Metric, F.Cu at (172.6, 76.4)
- added C24: 100nF, Capacitor_SMD:C_0603_1608Metric, F.Cu at (186.3, 64.7)
- added C3: 100nF, Capacitor_SMD:C_0603_1608Metric, F.Cu at (99.6, 71.7)
- added C4: 100nF, Capacitor_SMD:C_0603_1608Metric, F.Cu at (96.4, 87.8)
- added C5: 100nF, Capacitor_SMD:C_0603_1608Metric, F.Cu at (128.6, 70.8)
- added C6: 100nF, Capacitor_SMD:C_0603_1608Metric, F.Cu at (92.4, 87.8)
- added C7: 100nF, Capacitor_SMD:C_0603_1608Metric, F.Cu at (135.7, 67.6)
- added C8: 10uF, Capacitor_SMD:C_0603_1608Metric, F.Cu at (115.0, 88.0)
- added C9: 0.1uF, Capacitor_SMD:C_0603_1608Metric, F.Cu at (119.6, 84.1)
- added D1: WS2812B, LED_SMD:LED_WS2812B_PLCC4_5.0x5.0mm_P3.2mm, F.Cu at (176.1, 63.7)
- added D2: LED, LED_SMD:LED_0805_2012Metric, F.Cu at (182.5, 61.9)
- added D3: LED, LED_SMD:LED_0805_2012Metric, F.Cu at (172.8, 68.6)
- added D4: D_Schottky, Package_TO_SOT_SMD:SOT-23, F.Cu at (119.8, 80.5)
- added F1: 2A, Fuse:Fuse_1206_3216Metric_Castellated, F.Cu at (130.8, 62.0)
- added F2: 2A, Fuse:Fuse_1206_3216Metric_Castellated, F.Cu at (104.8, 85.4)
- added H1: MountingHole, MountingHole:MountingHole_2.2mm_M2_Pad_Via, F.Cu at (114.6, 81.2)
- added H2: MountingHole, MountingHole:MountingHole_2.2mm_M2_Pad_Via, F.Cu at (123.6, 70.2)
- added H3: MountingHole, MountingHole:MountingHole_2.2mm_M2_Pad_Via, F.Cu at (130.7, 66.5)
- added H4: MountingHole, MountingHole:MountingHole_2.2mm_M2_Pad_Via, F.Cu at (136.8, 63.3)
- added J1: Conn_01x02, TerminalBlock_Phoenix:TerminalBlock_Phoenix_PT-1,5-2-3.5-H_1x02_P3.50mm_Horizontal, F.Cu at (114.4, 72.7)
- added J2: USB_B_Micro, Connector_USB:USB_Micro-B_Molex_47346-0001, F.Cu at (102.8, 63.5)
- added J3: SWD, Connector_PinHeader_2.54mm:PinHeader_2x05_P2.54mm_Vertical, F.Cu at (92.7, 62.7)
- added J4: Micro_SD_Card, Connector_Card:microSD_HC_Hirose_DM3AT-SF-PEJM5, F.Cu at (153.1, 69.7)
- added J5: ST_01x02, TerminalBlock_Phoenix:TerminalBlock_Phoenix_PT-1,5-2-3.5-H_1x02_P3.50mm_Horizontal, F.Cu at (164.3, 71.3)
- added Q1: DMN2230U, Package_TO_SOT_SMD:SOT-23, F.Cu at (163.8, 79.1)
- added R1: 10K, Capacitor_SMD:C_0603_1608Metric, F.Cu at (136.6, 70.1)
- added R10: 150R, Capacitor_SMD:C_0603_1608Metric, F.Cu at (163.5, 82.6)
- added R11: 150R, Capacitor_SMD:C_0603_1608Metric, F.Cu at (182.3, 67.2)
- added R13: 10K, Capacitor_SMD:C_0603_1608Metric, F.Cu at (98.3, 101.1)
- added R14: 10K, Capacitor_SMD:C_0603_1608Metric, F.Cu at (102.7, 93.5)
- added R15: 200R, Capacitor_SMD:C_0603_1608Metric, F.Cu at (177.0, 68.2)
- added R16: 5R, Capacitor_SMD:C_0603_1608Metric, F.Cu at (172.6, 71.4)
- added R17: 100K, Capacitor_SMD:C_0603_1608Metric, F.Cu at (168.0, 78.0)
- added R18: 20K, Capacitor_SMD:C_0603_1608Metric, F.Cu at (182.3, 64.7)
- added R2: 10K, Capacitor_SMD:C_0603_1608Metric, F.Cu at (123.6, 84.1)
- added R3: 22R, Capacitor_SMD:C_0603_1608Metric, F.Cu at (119.0, 86.6)
- added R4: 100K, Capacitor_SMD:C_0603_1608Metric, F.Cu at (132.6, 73.3)
- added R5: 38K, Capacitor_SMD:C_0603_1608Metric, F.Cu at (128.5, 78.3)
- added R6: 22R, Capacitor_SMD:C_0603_1608Metric, F.Cu at (139.7, 67.6)
- added R7: 10K, Capacitor_SMD:C_0603_1608Metric, F.Cu at (128.6, 73.3)
- added R8: 150R, Capacitor_SMD:C_0603_1608Metric, F.Cu at (168.0, 80.5)
- added R9: 10K, Capacitor_SMD:C_0603_1608Metric, F.Cu at (172.6, 73.9)
- added SW1: SW_SPDT, Button_Switch_SMD:SW_SPDT_PCM12, F.Cu at (106.7, 79.8)
- added SW2: SW_SPDT, Button_Switch_SMD:SW_SPDT_PCM12, F.Cu at (122.8, 63.3)
- added SW3: SW_Push, Button_Switch_SMD:SW_SPST_B3U-1000P, F.Cu at (123.6, 75.4)
- added SW4: SW_Push, Button_Switch_SMD:SW_SPST_B3U-1000P, F.Cu at (93.3, 99.5)
- added TP1: TestPoint, TestPoint:TestPoint_Pad_D1.5mm, F.Cu at (127.4, 84.9)
- added TP2: TestPoint, TestPoint:TestPoint_Pad_D1.5mm, F.Cu at (132.3, 79.9)
- added TP3: TestPoint, TestPoint:TestPoint_Pad_D1.5mm, F.Cu at (122.8, 87.1)
- added TP4: TestPoint, TestPoint:TestPoint_Pad_D1.5mm, F.Cu at (136.4, 73.1)
- added TP5: TestPoint, TestPoint:TestPoint_Pad_D1.5mm, F.Cu at (127.8, 81.3)
- added TP6: TestPoint, TestPoint:TestPoint_Pad_D1.5mm, F.Cu at (132.3, 76.3)
- added U1: STM32F103C8Tx, Package_QFP:LQFP-48_7x7mm_P0.5mm, F.Cu at (96.1, 80.8)
- added U2: BMI088, BMI088:PQFN50P450X300X100-16N, F.Cu at (93.5, 95.0)
- added U3: LM1117-3.3, Package_TO_SOT_SMD:SOT-223, F.Cu at (106.7, 72.7)
- added U4: BMP280, Package_LGA:Bosch_LGA-8_2x2.5mm_P0.65mm_ClockwisePinNumbering, F.Cu at (98.6, 94.1)
- added U5: LM1117-3.3, Package_TO_SOT_SMD:SOT-223, F.Cu at (113.0, 64.5)
- added U6: W25Q32JVSS, Package_SO:SOIC-8_5.23x5.23mm_P1.27mm, F.Cu at (166.7, 63.7)
- added Y1: 16MHz, Crystal:Crystal_SMD_3225-4Pin_3.2x2.5mm, F.Cu at (110.4, 86.4)
