File: _autosave-OneAvionics.kicad_pcb (KiCad board)
At the start: 2 copper layers, 72 parts, among them J1 Conn_01x02, J2 USB_B_Micro, J3 SWD, J4 Micro_SD_Card, J5 ST_01x02, Q1 DMN2230U, SW1 SW_SPDT, SW2 SW_SPDT, SW3 SW_Push, SW4 SW_Push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

Commit message: more cleanup
Parts:
- removed C19: 100nF, Capacitor_SMD:C_0603_1608Metric
- removed R16: 5R, Capacitor_SMD:C_0603_1608Metric
- added C18: 100nF, Capacitor_SMD:C_0603_1608Metric, F.Cu at (237.7, 82.6)
- added R12: 4R, Resistor_SMD:R_0603_1608Metric, F.Cu at (214.9, 100.6)
- C23: footprint Capacitor_SMD:C_0603_1608Metric -> Capacitor_SMD:CP_Elec_10x10
- J1, J5: footprint TerminalBlock_Phoenix:TerminalBlock_Phoenix_PT-1,5-2-3.5-H_1x02_P3.50mm_Horizontal -> TerminalBlock:TerminalBlock_bornier-2_P5.08mm
- R1, R10, R11, R13, R14, R15, R17, R18, R2, R3, R4, R5, R6, R7, R9: footprint Capacitor_SMD:C_0603_1608Metric -> Resistor_SMD:R_0603_1608Metric
- R8: value 150R -> 50R; footprint Capacitor_SMD:C_0603_1608Metric -> Resistor_SMD:R_0603_1608Metric
- moved C16 127.3 mm to (233.7, 85.1)
- moved C13 66.3 mm to (149.7, 116.6)
- moved R9 65.8 mm to (238.2, 79.6)
- moved R10 61.2 mm to (224.0, 91.9)
- moved R8 60.7 mm to (228.0, 89.4)
- moved R13 58.2 mm to (153.7, 119.0)
- moved R17 57.2 mm to (224.0, 89.4)
- moved C15 56.8 mm to (158.1, 111.5)
- moved R14 55.3 mm to (154.1, 114.0)
- moved C1 54.5 mm to (179.9, 93.8)
- moved C10 54.5 mm to (184.0, 88.8)
- moved C11 54.5 mm to (175.4, 96.8)
- moved C2 54.5 mm to (175.4, 99.3)
- moved C22 54.5 mm to (151.0, 87.1)
- moved C3 54.5 mm to (151.0, 89.7)
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Connections:
- net +12V renamed +BATT
- net /RGB renamed /WS2812
- C16 pad 1: +3V3 -> GND
- C16 pad 2: GND -> +3V3
- C23 pad 1: GND -> Net-(C23-Pad1)
- C23 pad 2: Net-(C23-Pad2) -> GND
- J1 pad 1: Net-(D4-Pad2) -> GND
- J1 pad 2: GND -> Net-(D4-Pad2)
- J4 pad 2: /Output/CS_SD -> /CS_SD
- J5 pad 1: Net-(C23-Pad2) -> Net-(C23-Pad1)
- Q1 pad 2: Net-(Q1-Pad2) -> GND
- Q1 pad 3: Net-(J5-Pad2) -> Net-(Q1-Pad3)
- R15 pad 1: Net-(C23-Pad2) -> Net-(C23-Pad1)
- R17 pad 2: /Output/PYRO_CONT -> /PY1_CON
- R18 pad 1: /Output/PYRO_CONT -> /PY1_CON
- U1 pad 31: Net-(U1-Pad31) -> /PY1_CON
- U6 pad 1: /Output/CS_F -> /CS_FLASH
