File: OneAvionics.sch (KiCad schematic (older format))
At the start: 40 parts, among them J1 Conn_01x02, J2 USB_B_Micro, J3 SWD, SW1 SW_SPDT, SW2 SW_SPDT, SW3 SW_Push, U1 STM32F103C8Tx, U3 LM1117-3.3, Y1 16MHz

Commit message: rc and cont on pyro, linear reg, flash
Parts:
- removed R?: 10K, symbol Device:R_Small
- removed R?: 19.4K, symbol Device:R_Small
- added C?: 10uF, Capacitor_SMD:C_0603_1608Metric, symbol Device:C_Small
- added C?: 0.1uF, Capacitor_SMD:C_0603_1608Metric, symbol Device:C_Small
- added F?: 2A, Fuse:Fuse_1206_3216Metric_Castellated, symbol Device:Fuse
- added U?: LM1117-3.3, Package_TO_SOT_SMD:SOT-223, symbol Regulator_Linear:LM1117-3.3
- R4: value 10K -> 100K
- R5: value 3.8k -> 38K
Connections:
- net +3V3: now also C?.2, U?.2 (VO)
- net +5V: now also F?.2
- net GND: now also C?.1, C?.1, U?.1 (GND)
- new net: C?.2, F?.1, U?.3 (VI)
Other:
- note added: "LINEAR REG - 5V --> 3.3V"
- moved on the sheet: C3, C4, C5, C6, C7, R4, R5

Commit message: bno055 removed, bmi088, schotksy
Parts:
- added D4: D_Schottky, Package_TO_SOT_SMD:SOT-23, symbol Device:D_Schottky
- TP1, TP2, TP3, TP4, TP5, TP6: renamed from TP?; footprint (none) -> TestPoint:TestPoint_Pad_D1.5mm
- gave numbers to parts that had none: 4
Connections:
- net +12V: no longer J1.1 (Pin_1), SW2.2 (B)
- new net: D4.1 (K), SW2.2 (B)
- new net: D4.2 (A), J1.1 (Pin_1)
- no-connect marks 9 -> 5
Other:
- moved on the sheet: J1, SW2
Changed lines of the file:
@@
 F8 "LED" I L 7800 2100 39
-$EndSheet
-$Sheet
-S 3400 1250 1000 900
-U 604A6029
-F0 "Input" 39
-F1 "Input.sch" 39
-F2 "nBoot" I R 4400 1350 39
-F3 "INT" I R 4400 1475 39
-F4 "RESET" I R 4400 1600 39
-F5 "SDA" I R 4400 1725 39
-F6 "SCL" I R 4400 1850 39
-F7 "addr" I R 4400 1975 39
-F8 "BUTTON" I R 4400 2100 39
 $EndSheet
 Wire Notes Line
@@
 	3675 3375 3725 3375
 Connection ~ 3675 3375
-NoConn ~ 4400 1975
-NoConn ~ 4400 1600
-NoConn ~ 4400 1475
-NoConn ~ 4400 1350
 Text Label 5450 4000 2    39   ~ 0
 RGB
@@
 L power:GND #PWR0101
 U 1 1 6045EFB2
-P 8200 2825
-F 0 "#PWR0101" H 8200 2575 50  0001 C CNN
-F 1 "GND" V 8205 2697 50  0000 R CNN
-F 2 "" H 8200 2825 50  0001 C CNN
-F 3 "" H 8200 2825 50  0001 C CNN
-	1    8200 2825
+P 8300 2775
+F 0 "#PWR0101" H 8300 2525 50  0001 C CNN
+F 1 "GND" V 8305 2647 50  0000 R CNN
+F 2 "" H 8300 2775 50  0001 C CNN
+F 3 "" H 8300 2775 50  0001 C CNN
+	1    8300 2775
 	0    -1   -1   0
 $EndComp
@@
 L Connector_Generic:Conn_01x02 J1
 U 1 1 60459623
-P 8000 2925
-F 0 "J1" H 7918 2600 50  0000 C CNN
-F 1 "Conn_01x02" H 7918 2691 50  0000 C CNN
-F 2 "TerminalBlock_Phoenix:TerminalBlock_Phoenix_PT-1,5-2-3.5-H_1x02_P3.50mm_Horizontal" H 8000 2925 50  0001 C CNN
-F 3 "~" H 8000 2925 50  0001 C CNN
-	1    8000 2925
+P 8100 2875
+F 0 "J1" H 8018 2550 50  0000 C CNN
+F 1 "Conn_01x02" H 8018 2641 50  0000 C CNN
+F 2 "TerminalBlock_Phoenix:TerminalBlock_Phoenix_PT-1,5-2-3.5-H_1x02_P3.50mm_Horizontal" H 8100 2875 50  0001 C CNN
+F 3 "~" H 8100 2875 50  0001 C CNN
+	1    8100 2875
 	-1   0    0    1
-$EndComp
-$Comp
-L power:+12V #PWR0129
-U 1 1 605110C1
-P 8200 2925
-F 0 "#PWR0129" H 8200 2775 50  0001 C CNN
-F 1 "+12V" V 8215 3053 50  0000 L CNN
-F 2 "" H 8200 2925 50  0001 C CNN
-F 3 "" H 8200 2925 50  0001 C CNN
-	1    8200 2925
-	0    1    1    0
 $EndComp
 $Comp
 L power:+12V #PWR0110
 U 1 1 605FB599
-P 9500 2800
-F 0 "#PWR0110" H 9500 2650 50  0001 C CNN
-F 1 "+12V" V 9515 2928 50  0000 L CNN
-F 2 "" H 9500 2800 50  0001 C CNN
-F 3 "" H 9500 2800 50  0001 C CNN
-	1    9500 2800
+P 9375 2775
+F 0 "#PWR0110" H 9375 2625 50  0001 C CNN
+F 1 "+12V" V 9390 2903 50  0000 L CNN
+F 2 "" H 9375 2775 50  0001 C CNN
+F 3 "" H 9375 2775 50  0001 C CNN
+	1    9375 2775
 	0    1    1    0
 $EndComp
@@
 L Switch:SW_SPDT SW2
 U 1 1 60455D7B
-P 9300 2900
-F 0 "SW2" H 9300 3185 50  0000 C CNN
-F 1 "SW_SPDT" H 9300 3094 50  0000 C CNN
-F 2 "Button_Switch_SMD:SW_SPDT_PCM12" H 9300 2900 50  0001 C CNN
-F 3 "~" H 9300 2900 50  0001 C CNN
-	1    9300 2900
-	1    0    0    -1
-$EndComp
-NoConn ~ 9500 3000
-$Comp
-L power:+12V #PWR0130
-U 1 1 605114D9
-P 9100 2900
-F 0 "#PWR0130" H 9100 2750 50  0001 C CNN
-F 1 "+12V" V 9115 3028 50  0000 L CNN
-F 2 "" H 9100 2900 50  0001 C CNN
-F 3 "" H 9100 2900 50  0001 C CNN
-	1    9100 2900
-	0    -1   -1   0
-$EndComp
+P 9175 2875
+F 0 "SW2" H 9175 3160 50  0000 C CNN
+F 1 "SW_SPDT" H 9175 3069 50  0000 C CNN
+F 2 "Button_Switch_SMD:SW_SPDT_PCM12" H 9175 2875 50  0001 C CNN
+F 3 "~" H 9175 2875 50  0001 C CNN
+	1    9175 2875
+	1    0    0    -1
+$EndComp
+NoConn ~ 9375 2975
 Wire Wire Line
 	9200 3450 9200 3400
@@
 P 6875 5050
 AR Path="/604AFA5F/604B7FBC" Ref="TP?"  Part="1"
-AR Path="/604B7FBC" Ref="TP?"  Part="1"
-F 0 "TP?" V 7070 5122 50  0000 C CNN
+AR Path="/604B7FBC" Ref="TP3"  Part="1"
+F 0 "TP3" V 7070 5122 50  0000 C CNN
 F 1 "TestPoint" V 6979 5122 50  0000 C CNN
-F 2 "" H 7075 5050 50  0001 C CNN
+F 2 "TestPoint:TestPoint_Pad_D1.5mm" H 7075 5050 50  0001 C CNN
 F 3 "~" H 7075 5050 50  0001 C CNN
 	1    6875 5050
@@
 P 6875 5050
 AR Path="/604AFA5F/604B7FC2" Ref="#PWR?"  Part="1"
-AR Path="/604B7FC2" Ref="#PWR?"  Part="1"
-F 0 "#PWR?" H 6875 4900 50  0001 C CNN
+AR Path="/604B7FC2" Ref="#PWR0122"  Part="1"
+F 0 "#PWR0122" H 6875 4900 50  0001 C CNN
 F 1 "+3.3V" V 6890 5178 50  0000 L CNN
 F 2 "" H 6875 5050 50  0001 C CNN
@@
 P 7425 5050
 AR Path="/604AFA5F/604B7FC8" Ref="TP?"  Part="1"
-AR Path="/604B7FC8" Ref="TP?"  Part="1"
-F 0 "TP?" V 7620 5122 50  0000 C CNN
+AR Path="/604B7FC8" Ref="TP4"  Part="1"
+F 0 "TP4" V 7620 5122 50  0000 C CNN
 F 1 "TestPoint" V 7529 5122 50  0000 C CNN
-F 2 "" H 7625 5050 50  0001 C CNN
+F 2 "TestPoint:TestPoint_Pad_D1.5mm" H 7625 5050 50  0001 C CNN
 F 3 "~" H 7625 5050 50  0001 C CNN
 	1    7425 5050
@@
 P 7425 5050
 AR Path="/604AFA5F/604B7FCE" Ref="#PWR?"  Part="1"
-AR Path="/604B7FCE" Ref="#PWR?"  Part="1"
-F 0 "#PWR?" H 7425 4900 50  0001 C CNN
+AR Path="/604B7FCE" Ref="#PWR0139"  Part="1"
+F 0 "#PWR0139" H 7425 4900 50  0001 C CNN
 F 1 "+5V" V 7440 5178 50  0000 L CNN
 F 2 "" H 7425 5050 50  0001 C CNN
@@
 P 6850 5325
 AR Path="/604AFA5F/604B7FD4" Ref="TP?"  Part="1"
-AR Path="/604B7FD4" Ref="TP?"  Part="1"
-F 0 "TP?" V 7045 5397 50  0000 C CNN
+AR Path="/604B7FD4" Ref="TP1"  Part="1"
+F 0 "TP1" V 7045 5397 50  0000 C CNN
 F 1 "TestPoint" V 6954 5397 50  0000 C CNN
-F 2 "" H 7050 5325 50  0001 C CNN
+F 2 "TestPoint:TestPoint_Pad_D1.5mm" H 7050 5325 50  0001 C CNN
 F 3 "~" H 7050 5325 50  0001 C CNN
 	1    6850 5325
@@
 P 7425 5325
 AR Path="/604AFA5F/604B7FDA" Ref="TP?"  Part="1"
-AR Path="/604B7FDA" Ref="TP?"  Part="1"
-F 0 "TP?" V 7620 5397 50  0000 C CNN
+AR Path="/604B7FDA" Ref="TP5"  Part="1"
+F 0 "TP5" V 7620 5397 50  0000 C CNN
 F 1 "TestPoint" V 7529 5397 50  0000 C CNN
-F 2 "" H 7625 5325 50  0001 C CNN
+F 2 "TestPoint:TestPoint_Pad_D1.5mm" H 7625 5325 50  0001 C CNN
 F 3 "~" H 7625 5325 50  0001 C CNN
 	1    7425 5325
@@
 P 6850 5600
 AR Path="/604AFA5F/604BA055" Ref="TP?"  Part="1"
-AR Path="/604BA055" Ref="TP?"  Part="1"
-F 0 "TP?" V 7045 5672 50  0000 C CNN
+AR Path="/604BA055" Ref="TP2"  Part="1"
+F 0 "TP2" V 7045 5672 50  0000 C CNN
 F 1 "TestPoint" V 6954 5672 50  0000 C CNN
-F 2 "" H 7050 5600 50  0001 C CNN
+F 2 "TestPoint:TestPoint_Pad_D1.5mm" H 7050 5600 50  0001 C CNN
 F 3 "~" H 7050 5600 50  0001 C CNN
 	1    6850 5600
@@
 P 7425 5600
 AR Path="/604AFA5F/604BA6D7" Ref="TP?"  Part="1"
-AR Path="/604BA6D7" Ref="TP?"  Part="1"
-F 0 "TP?" V 7620 5672 50  0000 C CNN
+AR Path="/604BA6D7" Ref="TP6"  Part="1"
+F 0 "TP6" V 7620 5672 50  0000 C CNN
 F 1 "TestPoint" V 7529 5672 50  0000 C CNN
-F 2 "" H 7625 5600 50  0001 C CNN
+F 2 "TestPoint:TestPoint_Pad_D1.5mm" H 7625 5600 50  0001 C CNN
 F 3 "~" H 7625 5600 50  0001 C CNN
 	1    7425 5600
@@
 $EndComp
 $Comp
-L power:GND #PWR?
+L power:GND #PWR0140
 U 1 1 604C039D
 P 7425 5600
-F 0 "#PWR?" H 7425 5350 50  0001 C CNN
+F 0 "#PWR0140" H 7425 5350 50  0001 C CNN
 F 1 "GND" V 7430 5472 50  0000 R CNN
 F 2 "" H 7425 5600 50  0001 C CNN
@@
 	8600 4250 8600 4300
 $Comp
-L Device:C_Small C?
+L Device:C_Small C14
 U 1 1 605DAC91
 P 8600 4400
-F 0 "C?" H 8700 4375 50  0000 L CNN
+F 0 "C14" H 8700 4375 50  0000 L CNN
 F 1 "10uF" H 8691 4445 50  0000 L CNN
 F 2 "Capacitor_SMD:C_0603_1608Metric" H 8600 4400 50  0001 C CNN
@@
 $EndComp
 $Comp
-L Device:C_Small C?
+L Device:C_Small C22
 U 1 1 605DAC97
 P 9200 4400
-F 0 "C?" H 9108 4354 50  0000 R CNN
+F 0 "C22" H 9108 4354 50  0000 R CNN
 F 1 "0.1uF" H 9108 4445 50  0000 R CNN
 F 2 "Capacitor_SMD:C_0603_1608Metric" H 9200 4400 50  0001 C CNN
@@
 $EndComp
 $Comp
-L power:+3.3V #PWR?
+L power:+3.3V #PWR0141
 U 1 1 605DAC9D
 P 9500 4250
-F 0 "#PWR?" H 9500 4100 50  0001 C CNN
+F 0 "#PWR0141" H 9500 4100 50  0001 C CNN
 F 1 "+3.3V" V 9515 4378 50  0000 L CNN
 F 2 "" H 9500 4250 50  0001 C CNN
@@
 	9500 4250 9200 4250
 $Comp
-L power:GND #PWR?
+L power:GND #PWR0142
 U 1 1 605DACA5
 P 8900 4550
-F 0 "#PWR?" H 8900 4300 50  0001 C CNN
+F 0 "#PWR0142" H 8900 4300 50  0001 C CNN
 F 1 "GND" H 8905 4377 50  0000 C CNN
 F 2 "" H 8900 4550 50  0001 C CNN
@@
 	8900 4550 9200 4550
 $Comp
-L Device:Fuse F?
+L Device:Fuse F2
 U 1 1 605DACAE
 P 8325 4250
-F 0 "F?" V 8128 4250 50  0000 C CNN
+F 0 "F2" V 8128 4250 50  0000 C CNN
 F 1 "2A" V 8219 4250 50  0000 C CNN
 F 2 "Fuse:Fuse_1206_3216Metric_Castellated" V 8255 4250 50  0001 C CNN
@@
 	7800 4800 9900 4800
 $Comp
-L power:+5V #PWR?
+L power:+5V #PWR0143
 U 1 1 605E4445
 P 8175 4250
-F 0 "#PWR?" H 8175 4100 50  0001 C CNN
+F 0 "#PWR0143" H 8175 4100 50  0001 C CNN
 F 1 "+5V" V 8190 4378 50  0000 L CNN
 F 2 "" H 8175 4250 50  0001 C CNN
@@
 $EndComp
 $Comp
-L Regulator_Linear:LM1117-3.3 U?
+L Regulator_Linear:LM1117-3.3 U5
 U 1 1 605E5E28
 P 8900 4250
-F 0 "U?" H 8900 4492 50  0000 C CNN
+F 0 "U5" H 8900 4492 50  0000 C CNN
 F 1 "LM1117-3.3" H 8900 4401 50  0000 C CNN
 F 2 "Package_TO_SOT_SMD:SOT-223" H 8900 4250 50  0001 C CNN
@@
 Wire Notes Line
 	9900 2475 9900 6050
+$Comp
+L Device:D_Schottky D4
+U 1 1 605FF63E
+P 8825 2875
+F 0 "D4" H 8825 2658 50  0000 C CNN
+F 1 "D_Schottky" H 8825 2749 50  0000 C CNN
+F 2 "Package_TO_SOT_SMD:SOT-23" H 8825 2875 50  0001 C CNN
+F 3 "~" H 8825 2875 50  0001 C CNN
+	1    8825 2875
+	-1   0    0    1
+$EndComp
+Wire Wire Line
+	8675 2875 8300 2875
+$Sheet
+S 3400 1250 1000 900
+U 604A6029
+F0 "Input" 39
+F1 "Input.sch" 39
+F2 "BUTTON" I R 4400 2100 39
+F3 "SDA" I R 4400 1725 39
+F4 "SCL" I R 4400 1850 39
+$EndSheet
 $EndSCHEMATC

Commit message: Schematic cleanup, pyro
thanks ben for the advice
Parts:
- removed C1: 100nF, Capacitor_SMD:C_0603_1608Metric, symbol Device:C_Small
- added C?: 100nF, Capacitor_SMD:C_0603_1608Metric, symbol Device:C_Small
Connections:
- net +5V: now also C?.2
- net GND: now also J1.1 (Pin_1), C?.1; no longer J1.2 (Pin_2)
- net at D4.2 (A): now also J1.2 (Pin_2); no longer J1.1 (Pin_1)
- net +12V renamed +BATT
Other:
- note added: "LINEAR REG - 7.4V --> 3.3V"
- note removed: "LINEAR REG - 12V --> 3.3V"
- moved on the sheet: C2, C3, C4, C5, C6, C7, D4, J1, J3, R2, R7, SW2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

Commit message: more cleanup
Parts:
- J1: footprint TerminalBlock_Phoenix:TerminalBlock_Phoenix_PT-1,5-2-3.5-H_1x02_P3.50mm_Horizontal -> TerminalBlock:TerminalBlock_bornier-2_P5.08mm
- R1, R2, R3, R4, R6, R7: footprint Capacitor_SMD:C_0603_1608Metric -> Resistor_SMD:R_0603_1608Metric
- R5: value 38K -> 80K; footprint Capacitor_SMD:C_0603_1608Metric -> Resistor_SMD:R_0603_1608Metric
- gave numbers to parts that had none: 1
Connections:
- net PY1_CON: now reaches U1.31 (PA10)
- net RGB renamed WS2812
Other:
- moved on the sheet: F1, F2, R1, R2, SW1

Commit message: MOAR CLEANUP
Other:
- moved on the sheet: C10, C11, U1, Y1
