File: Hardware/Output.sch (KiCad schematic (older format))
At the start: 19 parts, among them J4 Micro_SD_Card, J5 ST_01x02, Q1 DMN2230U, U6 W25Q32JVSS

Commit message: added pdf
Parts:
- J5: footprint TerminalBlock:TerminalBlock_bornier-2_P5.08mm -> TerminalBlock_Phoenix:TerminalBlock_Phoenix_PT-1,5-2-3.5-H_1x02_P3.50mm_Horizontal
Changed lines of the file:
@@
 $Descr A4 11693 8268
 encoding utf-8
-Sheet 3 3
+Sheet 2 3
 Title ""
 Date ""
@@
 F 0 "J5" H 5955 3992 50  0000 L CNN
 F 1 "ST_01x02" H 5955 3901 50  0000 L CNN
-F 2 "TerminalBlock:TerminalBlock_bornier-2_P5.08mm" H 5875 4000 50  0001 C CNN
+F 2 "TerminalBlock_Phoenix:TerminalBlock_Phoenix_PT-1,5-2-3.5-H_1x02_P3.50mm_Horizontal" H 5875 4000 50  0001 C CNN
 F 3 "~" H 5875 4000 50  0001 C CNN
 	1    5875 4000
