File: Hardware/_autosave-OneAvionics.kicad_pcb (KiCad board)
At the start: 2 copper layers, 72 parts, among them J1 Conn_01x02, J2 USB_B_Micro, J3 SWD, J4 Micro_SD_Card, J5 ST_01x02, Q1 DMN2230U, SW1 SW_SPDT, SW2 SW_SPDT, SW3 SW_Push, SW4 SW_Push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

Commit message: added pdf
Parts:
- C23, J4: moved to B.Cu
- J1, J5: footprint TerminalBlock:TerminalBlock_bornier-2_P5.08mm -> TerminalBlock_Phoenix:TerminalBlock_Phoenix_PT-1,5-2-3.5-H_1x02_P3.50mm_Horizontal
- R5: value 38K -> 80K
- moved C23 142.4 mm to (80.8, 66.0)
- moved J4 134.4 mm to (81.3, 34.0)
- moved J5 132.5 mm to (83.8, 76.2)
- moved R1 125.7 mm to (69.7, 45.7)
- moved H1 122.8 mm to (66.0, 27.9)
- moved R2 118.7 mm to (69.7, 47.2)
- moved H3 116.3 mm to (66.0, 78.7)
- moved F1 113.5 mm to (69.5, 66.9), turned to 90 degrees
- moved SW3 112.8 mm to (68.5, 56.3), turned to 180 degrees
- moved SW2 109.3 mm to (65.6, 68.9), turned to 270 degrees
- moved SW1 106.6 mm to (65.7, 44.8), turned to 270 degrees
- moved D4 104.6 mm to (70.1, 71.5)
- moved R6 104.5 mm to (89.9, 59.7)
- moved Y1 101.9 mm to (74.3, 52.2), turned to 270 degrees
- moved H2 99.0 mm to (96.5, 27.9)
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Routing:
- net /BOOT0: track 0.00 -> 0.91 mm
- added copper zone on F.Cu, net +3V3
- added copper zone on B.Cu, net GND
Other:
- board outline added: 35.6 x 55.9 mm
